File: ltc3331-breakout.kicad_pcb (KiCad board)
At the start: 2 copper layers, 100 x 100 mm, 75 parts, among them IC1 LTC3331, J1 CONN_01X04, J10 CONN_01X02_FEMALE, J11 CONN_01X04, J12 CONN_01X03, J13 CONN_01X03, J14 CONN_01X03, J15 CONN_02X12, J16 CONN_02X08, J17 CONN_02X08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

Commit message: more cleanup
Parts:
- moved JP10 13.7 mm to (102.6, 130.0), turned to 180 degrees
- moved JP15 5.08 mm to (120.4, 82.9), turned to 0 degrees
- moved C7 3.06 mm to (102.6, 122.0), turned to 270 degrees
- moved JP4 2.62 mm to (98.6, 130.0), turned to 180 degrees
- moved JP11 2.33 mm to (107.8, 126.6)
- moved J20 2.16 mm to (58.8, 119.4)
- moved JP19 0.97 mm to (111.6, 126.6), turned to 180 degrees
- moved JP18 0.89 mm to (68.3, 78.2)
Routing:
- net GND: track 240.3 -> 229.9 mm, vias 41 -> 39
- net /BAT_IN: track 148.0 -> 155.1 mm
- net (no net): track 0.00 -> 5.72 mm, vias 0 -> 2
- net /SWB: track 28.3 -> 24.0 mm
- net /VIN: track 27.6 -> 30.4 mm
- net Net-(JP11-Pad1): track 15.3 -> 17.1 mm
- net Net-(JP19-Pad1): track 22.2 -> 20.8 mm
- net Net-(C1-Pad2): track 5.02 -> 3.62 mm
- net /BAL: track 133.1 -> 134.0 mm
Other:
- board text added: "22uH SWA-SWB"
- board text added: "22uH VOUT-SW"
- board text added: "CHARGE CURRENT RESISTOR"
- board text removed: "22uH SW/VOUT"
- board text removed: "22uH SWA/SWB"
- board text removed: "CHRG CURNT RES"
